File: splembedded.kicad_pcb (KiCad board)
At the start: 2 copper layers, 140 x 81.3 mm, 30 parts, among them SW1 Switch, SW10 Switch, SW11 Switch, SW12 Switch, SW13 Switch, SW14 Switch, SW15 Switch, SW2 Switch, SW3 Switch, SW4 Switch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

Commit message: smd branch init
Parts:
- removed the display* at (186.3, 130.5)
- added J3: Pin Connector, Connector_PinSocket_2.54mm:PinSocket_1x02_P2.54mm_Vertical, F.Cu at (105.9, 148.5)
- added J4: JST Connector, Connector_JST:JST_PH_S2B-PH-K_1x02_P2.00mm_Horizontal, F.Cu at (109.6, 147.9)
- added RF*: JP, Jumper:SolderJumper-2_P1.3mm_Open_TrianglePad1.0x1.5mm, F.Cu at (182.4, 146.1)
- added RF*: JP, Jumper:SolderJumper-2_P1.3mm_Open_TrianglePad1.0x1.5mm, F.Cu at (192.6, 146.1)
- added RF*: JP, Jumper:SolderJumper-2_P1.3mm_Open_TrianglePad1.0x1.5mm, F.Cu at (185.0, 146.1)
- added RF*: JP, Jumper:SolderJumper-2_P1.3mm_Open_TrianglePad1.0x1.5mm, F.Cu at (190.1, 146.1)
- added RF*: JP, Jumper:SolderJumper-2_P1.3mm_Open_TrianglePad1.0x1.5mm, B.Cu at (190.1, 146.1)
- added RF*: JP, Jumper:SolderJumper-2_P1.3mm_Open_TrianglePad1.0x1.5mm, B.Cu at (192.6, 146.1)
- added RF*: JP, Jumper:SolderJumper-2_P1.3mm_Open_TrianglePad1.0x1.5mm, B.Cu at (185.0, 146.1)
- added RF*: JP, Jumper:SolderJumper-2_P1.3mm_Open_TrianglePad1.0x1.5mm, B.Cu at (182.4, 146.1)
- added SW2: SW_SPST, MSK-12C02:MSK-12C02, F.Cu at (87.5, 100.8)
- added SW2: SW_SPST, MSK-12C02:MSK-12C02, B.Cu at (87.5, 100.8)
- U1, U2: value xiao-ble -> xiao-ble-thruhole; footprint footprints:xiao-ble -> mcu:xiao-ble-smd-cutout
- moved U1 2.92 mm to (188.8, 100.3)
- moved U2 0.90 mm to (188.8, 100.3)
Connections:
- display* pad 1: COPI -> LCD_JP0
- display* pad 2: SCK -> LCD_JP1
- display* pad 4: GND -> LCD_JP2
- display* pad 5: LCD_CS -> LCD_JP3
Routing:
- net BAT+: track 0.00 -> 135.6 mm, vias 0 -> 3
- net GND: track 144.2 -> 10.6 mm, vias 3 -> 30
- net VBAT: track 0.00 -> 59.7 mm, vias 0 -> 3
- net R2: track 150.1 -> 188.4 mm, vias 0 -> 1
- net 3V3: track 136.8 -> 102.8 mm
- net R1: track 140.5 -> 172.9 mm, vias 0 -> 1
- net R0: track 136.9 -> 158.0 mm, vias 0 -> 1
- net COPI: track 105.2 -> 86.6 mm, vias 2 -> 3
- net LCD_CS: track 83.8 -> 66.3 mm, vias 1 -> 2
- net R3: track 101.9 -> 118.4 mm, vias 0 -> 1
- net FLASH_CS: track 30.5 -> 46.8 mm
- net SCK: track 90.4 -> 79.2 mm, vias 2 -> 3
- net CIPO: track 37.2 -> 32.6 mm
- net LCD_JP3: track 0.00 -> 4.12 mm
- net LCD_JP2: track 0.00 -> 4.12 mm
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- added copper zone on B.Cu, net GND
- added copper zone on F.Cu, net GND
Other:
- board size 140 x 81.3 mm -> 156.1 x 94.3 mm

Commit message: progress
Parts:
- added SW18: SW_Push, kbd:ResetSW, F.Cu at (96.4, 97.9)
- U1, U2: footprint mcu:xiao-ble-smd-cutout -> mcu:xiao-ble-smd
- moved J4 19.8 mm to (128.2, 141.4), turned to 0 degrees
- moved J3 18.5 mm to (123.9, 144.3), turned to 180 degrees
Routing:
- net RESET: track 0.00 -> 104.1 mm
- net VBAT: track 59.7 -> 143.3 mm, vias 3 -> 0
- net R0: track 158.0 -> 153.9 mm, vias 1 -> 2
- net BAT+: track 135.6 -> 139.0 mm
- net 3V3: track 102.8 -> 101.2 mm
- net LCD_CS: track 66.3 -> 65.2 mm
- net GND: vias 30 -> 33

Commit message: fix vbat trace
Routing:
- net VBAT: track 143.3 -> 145.0 mm, vias 0 -> 1
Changed lines of the file:
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@@
   (segment (start 123.916993 141.79101) (end 124.925983 142.8) (width 0.4) (layer "F.Cu") (net 24))
   (segment (start 128.88 142.8) (end 129.92 141.76) (width 0.4) (layer "F.Cu") (net 24))
+  (segment (start 88.70163 102.642999) (end 87.091599 102.985221) (width 0.4) (layer "F.Cu") (net 24))
+  (via (at 88.70163 102.642999) (size 0.4) (drill 0.2) (layers "F.Cu" "B.Cu") (net 24))
   (segment (start 105.755362 145.963182) (end 97.394293 154.324251) (width 0.4) (layer "B.Cu") (net 24))
   (segment (start 68.062 110.148) (end 61.53 114.85) (width 0.4) (layer "B.Cu") (net 24))
